Commit message: chassis urdf aint easy lol

File: src/chassisv003/urdf/chassisv003.urdf (robot description, URDF)
Before this commit: robot chassisv003, 18 links, 17 joints
Links:
- link chassis_link: geometry collision mesh filename=package://rover_description/meshes/Chassis_Frame.STL; visual mesh filename=package://rover_description/meshes/Chassis_Frame.STL
- link left_bogie_link: geometry collision mesh filename=package://rover_description/meshes/left_bogie_link.STL; visual mesh filename=package://rover_description/meshes/left_bogie_link.STL
- link rear_bogie_link: geometry collision mesh filename=package://rover_description/meshes/back_bogie_link.STL; visual mesh filename=package://rover_description/meshes/back_bogie_link.STL
- link right_bogie_link: geometry collision mesh filename=package://rover_description/meshes/right_bogie_link.STL; visual mesh filename=package://rover_description/meshes/right_bogie_link.STL
Joints:
- joint J1: axis 0 0 0 -> 0 0 1
- joint J2: axis 0 0 0 -> 1 0 0; origin xyz=0.1255 -0.050208 0.25442 rpy=2.1053 0 0.63509 -> xyz=0.065 0.055 0.11 rpy=2.1053 0 0.63509
- joint J3: axis 0 0 0 -> 1 0 0
- joint J4: axis 0 0 0 -> 1 0 0
- joint J5: axis 0 0 0 -> 0 1 0
- joint J6: axis 0 0 0 -> 0 0 1
