Commit message: gz start unpaused

File: src/Full_Assembly/urdf/Full_Assembly.urdf (robot description, URDF)
Before this commit: robot Full_Assembly, 15 links, 14 joints
Links:
- removed link Axis_1
- removed link Axis_2
- removed link Axis_3
- removed link Axis_4
Joints:
- removed joint J1
- removed joint J2
- removed joint J3
- removed joint J4
- joint Back_Connect: type fixed -> continuous
- joint Left_Connect: axis 0 0 0.999995325686932 -> 0 0 1; type fixed -> continuous
- joint Right_Connect: type fixed -> continuous
