Commit message: got arm locked to world

File: src/snowbots_arm_urdf_simplified_v5_12/urdf/snowbots_arm_urdf_simplified_v5_12.urdf (robot description, URDF)
Before this commit: robot snowbots_arm_urdf_simplified_v5_12, 8 links, 7 joints
Links:
- added link world
Joints:
- added joint world_joint: type fixed, parent world, child l1, origin xyz=-0.16681 -0.11566 0.018262 rpy=0 0 0, axis 0 0 1

Commit message: changed urdf inertia tags changed around what controllers launch -> from all three to just effort_controller arm is just slamming down as soon as controllers start, might be with the axis ranges

File: src/snowbots_arm_urdf_simplified_v5_12/urdf/snowbots_arm_urdf_simplified_v5_12.urdf (robot description, URDF)
Before this commit: robot snowbots_arm_urdf_simplified_v5_12, 9 links, 8 joints
Joints:
- joint world_joint: axis 0 0 1 -> (none); origin xyz=-0.16681 -0.11566 0.018262 rpy=0 0 0 -> xyz=0.0 0.0 0.0 rpy=0 0 0

Commit message: got test_old_urdf demo_gazebo.launch working to an extent pid values need tuning, and base is all wobbly also need a new urdf

File: src/snowbots_arm_urdf_simplified_v5_12/urdf/snowbots_arm_urdf_simplified_v5_12.urdf (robot description, URDF)
Before this commit: robot snowbots_arm_urdf_simplified_v5_12, 9 links, 8 joints
Links:
- link l3: mass 1.02884531575438 -> 0.102884531575438
Joints:
- joint j3: limit (none) -> lower=-1.13446 upper=1.13446 effort=30.0 velocity=1.0; type continuous -> revolute
- joint j7: axis 0 0 0 -> (none)
- joint world_joint: axis (none) -> 0 0 1

Commit message: added camera and custom world file

File: src/snowbots_arm_urdf_simplified_v5_12/urdf/snowbots_arm_urdf_simplified_v5_12.urdf (robot description, URDF)
Before this commit: robot snowbots_arm_urdf_simplified_v5_12, 9 links, 8 joints
Links:
- added link camera_link, mass 0.1
Joints:
- added joint camera_joint: type fixed, parent ef, child camera_link, origin xyz=0 0 0.2 rpy=0 0 1
- joint world_joint: origin xyz=0.0 0.0 0.0 rpy=0 0 0 -> xyz=0.0 0.0 1.09 rpy=0 0 0
