Commit message: just in case

File: src/rover_gazebo/urdf/minirover4.urdf (robot description, URDF)
Before this commit: robot minirover4, 10 links, 9 joints
Links:
- removed link linkt_right
- added link link_right, mass 1.7536; collision mesh filename=package://minirover4/meshes/link_right.STL; visual mesh filename=package://minirover4/meshes/link_right.STL
Joints:
- joint joint_frontright: parent linkt_right -> link_right
- joint joint_midright: parent linkt_right -> link_right
- joint joint_right: child linkt_right -> link_right
